File: CurrentSinkOrSwim.sch (KiCad schematic (older format))
At the start: 0 parts

Commit message: Added inital placements of components onto the PCB
Parts:
- added Q?: MOSFET_P, symbol MOSFET_P
- added R? (x2): R, symbol R
- added RV?: POT, symbol POT
- added U?: LM358, symbol LM358
- added U?: TC1016, symbol TC1016
Connections:
- net labels added: GND
- wire segments 0 -> 24
Changed lines of the file:
@@
 LIBS:contrib
 LIBS:valves
+LIBS:CustomComponents
+LIBS:CurrentSinkOrSwim-cache
 EELAYER 25 0
 EELAYER END
@@
 Comment4 ""
 $EndDescr
+$Comp
+L LM358 U?
+U 1 1 54CE7078
+P 5250 3050
+F 0 "U?" H 5200 3250 60  0000 L CNN
+F 1 "LM358" H 5200 2800 60  0000 L CNN
+F 2 "" H 5250 3050 60  0000 C CNN
+F 3 "" H 5250 3050 60  0000 C CNN
+	1    5250 3050
+	1    0    0    -1
+$EndComp
+$Comp
+L TC1016 U?
+U 1 1 54CE7607
+P 4500 1850
+F 0 "U?" H 4650 1450 60  0000 C CNN
+F 1 "TC1016" H 4500 2050 60  0000 C CNN
+F 2 "" H 4500 1850 60  0000 C CNN
+F 3 "" H 4500 1850 60  0000 C CNN
+	1    4500 1850
+	1    0    0    -1
+$EndComp
+$Comp
+L R R?
+U 1 1 54CE76B8
+P 4250 4100
+F 0 "R?" V 4330 4100 50  0000 C CNN
+F 1 "R" V 4257 4101 50  0000 C CNN
+F 2 "" V 4180 4100 30  0000 C CNN
+F 3 "" H 4250 4100 30  0000 C CNN
+	1    4250 4100
+	1    0    0    -1
+$EndComp
+$Comp
+L R R?
+U 1 1 54CE7735
+P 6400 4100
+F 0 "R?" V 6480 4100 50  0000 C CNN
+F 1 "R" V 6407 4101 50  0000 C CNN
+F 2 "" V 6330 4100 30  0000 C CNN
+F 3 "" H 6400 4100 30  0000 C CNN
+	1    6400 4100
+	1    0    0    -1
+$EndComp
+$Comp
+L MOSFET_P Q?
+U 1 1 54CE777E
+P 6300 3050
+F 0 "Q?" H 6300 3240 50  0000 R CNN
+F 1 "MOSFET_P" H 6300 2870 50  0000 R CNN
+F 2 "" H 6300 3050 60  0000 C CNN
+F 3 "" H 6300 3050 60  0000 C CNN
+	1    6300 3050
+	1    0    0    -1
+$EndComp
+Wire Wire Line
+	5750 3050 6100 3050
+Wire Wire Line
+	6400 3250 6400 3650
+Wire Wire Line
+	6400 3650 6400 3850
+Wire Wire Line
+	4900 2100 5150 2100
+Wire Wire Line
+	5150 2100 5150 2500
+Wire Wire Line
+	5150 2500 5150 2650
+Wire Wire Line
+	5150 2500 4250 2500
+Wire Wire Line
+	4250 2500 4250 2700
+Connection ~ 5150 2500
+Wire Wire Line
+	4250 3200 4250 3850
+$Comp
+L POT RV?
+U 1 1 54CE7B4E
+P 4250 2950
+F 0 "RV?" H 4250 2850 50  0000 C CNN
+F 1 "POT" H 4250 2950 50  0000 C CNN
+F 2 "" H 4250 2950 60  0000 C CNN
+F 3 "" H 4250 2950 60  0000 C CNN
+	1    4250 2950
+	0    1    1    0
+$EndComp
+Wire Wire Line
+	4400 2950 4550 2950
+Wire Wire Line
+	4550 2950 4750 2950
+Wire Wire Line
+	4550 2950 4550 4350
+Wire Wire Line
+	4550 4350 5150 4350
+Wire Wire Line
+	5150 4350 6400 4350
+Connection ~ 4550 2950
+$Comp
+L GND #PWR?
+U 1 1 54CE7C2D
+P 6400 4500
+F 0 "#PWR?" H 6400 4250 60  0001 C CNN
+F 1 "GND" H 6400 4350 60  0000 C CNN
+F 2 "" H 6400 4500 60  0000 C CNN
+F 3 "" H 6400 4500 60  0000 C CNN
+	1    6400 4500
+	1    0    0    -1
+$EndComp
+$Comp
+L GND #PWR?
+U 1 1 54CE7C41
+P 4250 4550
+F 0 "#PWR?" H 4250 4300 60  0001 C CNN
+F 1 "GND" H 4250 4400 60  0000 C CNN
+F 2 "" H 4250 4550 60  0000 C CNN
+F 3 "" H 4250 4550 60  0000 C CNN
+	1    4250 4550
+	1    0    0    -1
+$EndComp
+$Comp
+L GND #PWR?
+U 1 1 54CE7C55
+P 3900 2250
+F 0 "#PWR?" H 3900 2000 60  0001 C CNN
+F 1 "GND" H 3900 2100 60  0000 C CNN
+F 2 "" H 3900 2250 60  0000 C CNN
+F 3 "" H 3900 2250 60  0000 C CNN
+	1    3900 2250
+	1    0    0    -1
+$EndComp
+Wire Wire Line
+	4100 2100 3900 2100
+Wire Wire Line
+	3900 2100 3900 2250
+Wire Wire Line
+	4250 4350 4250 4550
+Wire Wire Line
+	6400 4350 6400 4500
+Wire Wire Line
+	5150 3450 5150 4350
+Connection ~ 5150 4350
+Wire Wire Line
+	4750 3150 4750 3650
+Wire Wire Line
+	4750 3650 6400 3650
+Connection ~ 6400 3650
+Wire Wire Line
+	4900 1800 6400 1800
+Wire Wire Line
+	6400 1800 6900 1800
+Wire Wire Line
+	6400 1800 6400 2850
+Connection ~ 6400 1800
 $EndSCHEMATC
