File: CurrentSinkOrSwim.sch (KiCad schematic (older format))
At the start: 3 parts, among them P101 CONN_01X03, P102 CONN_01X02, P103 CONN_01X02

Commit message: Routing and fixing schematic checkpoint
Other:
- note added: "Sheet 200 Series"
- note added: "Sheet 300 Series"
- note added: "Sheet 400 Series"
Changed lines of the file:
@@
 	2550 1650 5150 1650
 $Comp
-L GND #PWR01
+L GND #PWR101
 U 1 1 54E393D4
 P 2700 2150
-F 0 "#PWR01" H 2700 1900 60  0001 C CNN
+F 0 "#PWR101" H 2700 1900 60  0001 C CNN
 F 1 "GND" H 2700 2000 60  0000 C CNN
 F 2 "" H 2700 2150 60  0000 C CNN
@@
 	3200 5600 3600 5600
 $Comp
-L GND #PWR02
+L GND #PWR102
 U 1 1 54E3C230
 P 5900 6550
-F 0 "#PWR02" H 5900 6300 60  0001 C CNN
+F 0 "#PWR102" H 5900 6300 60  0001 C CNN
 F 1 "GND" H 5900 6400 60  0000 C CNN
 F 2 "" H 5900 6550 60  0000 C CNN
@@
 Wire Wire Line
 	5900 4150 4950 4150
+Text Notes 2950 2800 0    60   ~ 0
+Sheet 400 Series
+Text Notes 2750 3500 0    60   ~ 0
+Sheet 200 Series
+Text Notes 2700 6400 0    60   ~ 0
+Sheet 300 Series
 $EndSCHEMATC

Commit message: Initial route before filling the ground plane
Changed lines of the file:
@@
 	2550 1650 5150 1650
 $Comp
-L GND #PWR101
+L GND #PWR01
 U 1 1 54E393D4
 P 2700 2150
-F 0 "#PWR101" H 2700 1900 60  0001 C CNN
+F 0 "#PWR01" H 2700 1900 60  0001 C CNN
 F 1 "GND" H 2700 2000 60  0000 C CNN
 F 2 "" H 2700 2150 60  0000 C CNN
@@
 $EndSheet
 $Sheet
-S 3600 5250 1400 1200
+S 2150 5250 1400 1200
 U 54E38475
 F0 "Voltage Control" 60
 F1 "VoltageControl.sch" 60
-F2 "Vcontrol" O L 3600 5600 60
-F3 "Current_Sink+" I R 5000 5550 60
-F4 "Current_Sink-" I R 5000 5950 60
+F2 "Vcontrol" O L 2150 5600 60
+F3 "Current_Sink+" I R 3550 5550 60
+F4 "Current_Sink-" I R 3550 5950 60
 $EndSheet
 $Sheet
@@
 	5250 1550 5250 2150
 Wire Wire Line
-	5350 5550 5000 5550
+	5350 5550 3550 5550
 Connection ~ 5350 3600
 Wire Wire Line
-	5900 5950 5000 5950
+	5900 5950 3550 5950
 Connection ~ 5900 4150
 Wire Wire Line
-	3600 4000 3200 4000
+	3600 4000 1650 4000
 Wire Wire Line
-	3200 4000 3200 5600
+	1650 4000 1650 5600
 Wire Wire Line
-	3200 5600 3600 5600
+	1650 5600 2150 5600
 $Comp
-L GND #PWR102
+L GND #PWR02
 U 1 1 54E3C230
 P 5900 6550
-F 0 "#PWR102" H 5900 6300 60  0001 C CNN
+F 0 "#PWR02" H 5900 6300 60  0001 C CNN
 F 1 "GND" H 5900 6400 60  0000 C CNN
 F 2 "" H 5900 6550 60  0000 C CNN

Commit message: Final update to BOM and added the bom XSL script
Parts:
- P101: MPN (none) -> M20-9990346
- P102, P103: MPN (none) -> 50500020134G
Changed lines of the file:
@@
 F 2 "CSOS Local:Terminal_Block_1x200_mil" H 6250 2400 60  0001 C CNN
 F 3 "" H 6250 2400 60  0000 C CNN
+F 4 "50500020134G" H 6250 2400 60  0001 C CNN "MPN"
 	1    6250 2400
 	1    0    0    -1
@@
 F 2 "Pin_Headers:Pin_Header_Straight_1x03" H 5250 1350 60  0001 C CNN
 F 3 "" H 5250 1350 60  0000 C CNN
+F 4 "M20-9990346" H 5250 1350 60  0001 C CNN "MPN"
 	1    5250 1350
 	0    -1   -1   0
@@
 F 2 "CSOS Local:Terminal_Block_1x200_mil" H 2350 1700 60  0001 C CNN
 F 3 "" H 2350 1700 60  0000 C CNN
+F 4 "50500020134G" H 2350 1700 60  0001 C CNN "MPN"
 	1    2350 1700
 	-1   0    0    -1
