File: VoltageControl.sch (KiCad schematic (older format))
At the start: 7 parts

Commit message: Initial annotation
Parts:
- R301, R302, R303: renamed from R?; footprint (none) -> Resistors_SMD:R_0603_HandSoldering
- U201: renamed from U?; footprint (none) -> SMD_Packages:SSOP-8
- gave numbers to parts that had none: 3
Connections:
- wire segments 26 -> 21
Changed lines of the file:
@@
 $EndDescr
 $Comp
-L LMV358 U?
-U 1 1 54E398B3
+L LMV358 U201
+U 2 1 54E398B3
 P 5500 2750
-F 0 "U?" H 5450 2950 60  0000 L CNN
+F 0 "U201" H 5450 2950 60  0000 L CNN
 F 1 "LMV358" H 5450 2500 60  0000 L CNN
-F 2 "" H 5500 2750 60  0000 C CNN
+F 2 "SMD_Packages:SSOP-8" H 5500 2750 60  0001 C CNN
 F 3 "" H 5500 2750 60  0000 C CNN
-	1    5500 2750
+	2    5500 2750
 	1    0    0    -1
 $EndComp
 $Comp
-L DIODE D?
+L DIODE D301
 U 1 1 54E3AD95
 P 6450 2750
-F 0 "D?" H 6450 2850 50  0000 C CNN
+F 0 "D301" H 6450 2850 50  0000 C CNN
 F 1 "DIODE" H 6450 2650 50  0000 C CNN
-F 2 "" H 6450 2750 60  0000 C CNN
+F 2 "" H 6450 2750 60  0001 C CNN
 F 3 "" H 6450 2750 60  0000 C CNN
 	1    6450 2750
@@
 $EndComp
 $Comp
-L R R?
+L R R302
 U 1 1 54E3B0B9
 P 4150 3550
-F 0 "R?" V 4230 3550 50  0000 C CNN
+F 0 "R302" V 4230 3550 50  0000 C CNN
 F 1 "R" V 4157 3551 50  0000 C CNN
-F 2 "" V 4080 3550 30  0000 C CNN
+F 2 "Resistors_SMD:R_0603_HandSoldering" V 4080 3550 30  0001 C CNN
 F 3 "" H 4150 3550 30  0000 C CNN
 	1    4150 3550
@@
 $EndComp
 $Comp
-L C C?
+L C C301
 U 1 1 54E3B0CD
 P 5000 2050
-F 0 "C?" H 5050 2150 50  0000 L CNN
+F 0 "C301" H 5050 2150 50  0000 L CNN
 F 1 "C" H 5050 1950 50  0000 L CNN
-F 2 "" H 5038 1900 30  0000 C CNN
+F 2 "" H 5038 1900 30  0001 C CNN
 F 3 "" H 5000 2050 60  0000 C CNN
 	1    5000 2050
@@
 $EndComp
 Wire Wire Line
-	4150 3100 4150 3200
-Wire Wire Line
-	4150 3200 4150 3300
+	4150 3100 4150 3300
 Wire Wire Line
 	4150 3800 4150 4550
@@
 	4800 2850 4800 3700
 $Comp
-L POT RV?
+L POT RV301
 U 1 1 54E3B0DA
 P 4150 2850
-F 0 "RV?" H 4150 2750 50  0000 C CNN
+F 0 "RV301" H 4150 2750 50  0000 C CNN
 F 1 "POT" H 4150 2850 50  0000 C CNN
-F 2 "" H 4150 2850 60  0000 C CNN
+F 2 "" H 4150 2850 60  0001 C CNN
 F 3 "" H 4150 2850 60  0000 C CNN
 	1    4150 2850
@@
 	5400 1750 5400 2350
 Wire Wire Line
-	3900 1750 4400 1750
-Wire Wire Line
-	4400 1750 5000 1750
-Wire Wire Line
-	5000 1750 5400 1750
+	3900 1750 5400 1750
 Connection ~ 4400 1750
 Wire Wire Line
@@
 	6650 2750 7250 2750
 $Comp
-L R R?
+L R R301
 U 1 1 54E3B1F8
 P 6100 3350
-F 0 "R?" V 6180 3350 50  0000 C CNN
+F 0 "R301" V 6180 3350 50  0000 C CNN
 F 1 "9K" V 6107 3351 50  0000 C CNN
-F 2 "" V 6030 3350 30  0000 C CNN
+F 2 "Resistors_SMD:R_0603_HandSoldering" V 6030 3350 30  0001 C CNN
 F 3 "" H 6100 3350 30  0000 C CNN
 	1    6100 3350
@@
 $EndComp
 $Comp
-L R R?
+L R R303
 U 1 1 54E3B24B
 P 6100 4150
-F 0 "R?" V 6180 4150 50  0000 C CNN
+F 0 "R303" V 6180 4150 50  0000 C CNN
 F 1 "1K" V 6107 4151 50  0000 C CNN
-F 2 "" V 6030 4150 30  0000 C CNN
+F 2 "Resistors_SMD:R_0603_HandSoldering" V 6030 4150 30  0001 C CNN
 F 3 "" H 6100 4150 30  0000 C CNN
 	1    6100 4150
@@
 	6100 4400 6100 4550
 Wire Wire Line
-	4150 4550 6100 4550
-Wire Wire Line
-	6100 4550 7250 4550
+	4150 4550 7250 4550
 Text HLabel 7250 2750 2    60   Output ~ 0
 Vcontrol
@@
 	4800 3700 6100 3700
 Wire Wire Line
-	6100 3600 6100 3700
-Wire Wire Line
-	6100 3700 6100 3900
+	6100 3600 6100 3900
 Connection ~ 6100 3700
 Wire Wire Line

Commit message: Preliminary footprint association
Parts:
- C301: footprint (none) -> SMD_Packages:SMD-0805
- D301: footprint (none) -> SMD_Packages:SOD-523; MPN (none) -> 1N4148WT
- R301, R302, R303: footprint Resistors_SMD:R_0603_HandSoldering -> SMD_Packages:SMD-0805
- RV301: footprint (none) -> Potentiometers:Potentiometer_WirePads_largePads
- U201: footprint SMD_Packages:SSOP-8 -> SMD_Packages:SOIC-8-N; MPN (none) -> LMV358IDR
Changed lines of the file:
@@
 F 0 "U201" H 5450 2950 60  0000 L CNN
 F 1 "LMV358" H 5450 2500 60  0000 L CNN
-F 2 "SMD_Packages:SSOP-8" H 5500 2750 60  0001 C CNN
-F 3 "" H 5500 2750 60  0000 C CNN
+F 2 "SMD_Packages:SOIC-8-N" H 5500 2750 60  0001 C CNN
+F 3 "http://www.produktinfo.conrad.com/datenblaetter/1000000-1099999/001072383-da-01-en-IC_OPAMP_GP_R_R_1MH_LMV358IDR_SOIC_8_TID.pdf" H 5500 2750 60  0001 C CNN
+F 4 "LMV358IDR" H 5500 2750 60  0001 C CNN "MPN"
 	2    5500 2750
 	1    0    0    -1
@@
 F 0 "D301" H 6450 2850 50  0000 C CNN
 F 1 "DIODE" H 6450 2650 50  0000 C CNN
-F 2 "" H 6450 2750 60  0001 C CNN
-F 3 "" H 6450 2750 60  0000 C CNN
+F 2 "SMD_Packages:SOD-523" H 6450 2750 60  0001 C CNN
+F 3 "http://www.conrad.de/ce/de/product/1262771/Diode-Fairchild-Semiconductor-1N4148WT-Gehaeuseart-SOD-523-F?ref=searchDetail" H 6450 2750 60  0001 C CNN
+F 4 "1N4148WT" H 6450 2750 60  0001 C CNN "MPN"
 	1    6450 2750
 	-1   0    0    1
@@
 F 0 "R302" V 4230 3550 50  0000 C CNN
 F 1 "R" V 4157 3551 50  0000 C CNN
-F 2 "Resistors_SMD:R_0603_HandSoldering" V 4080 3550 30  0001 C CNN
+F 2 "SMD_Packages:SMD-0805" V 4080 3550 30  0001 C CNN
 F 3 "" H 4150 3550 30  0000 C CNN
 	1    4150 3550
@@
 F 0 "C301" H 5050 2150 50  0000 L CNN
 F 1 "C" H 5050 1950 50  0000 L CNN
-F 2 "" H 5038 1900 30  0001 C CNN
+F 2 "SMD_Packages:SMD-0805" H 5038 1900 30  0001 C CNN
 F 3 "" H 5000 2050 60  0000 C CNN
 	1    5000 2050
@@
 F 0 "RV301" H 4150 2750 50  0000 C CNN
 F 1 "POT" H 4150 2850 50  0000 C CNN
-F 2 "" H 4150 2850 60  0001 C CNN
+F 2 "Potentiometers:Potentiometer_WirePads_largePads" H 4150 2850 60  0001 C CNN
 F 3 "" H 4150 2850 60  0000 C CNN
 	1    4150 2850
@@
 F 0 "R301" V 6180 3350 50  0000 C CNN
 F 1 "9K" V 6107 3351 50  0000 C CNN
-F 2 "Resistors_SMD:R_0603_HandSoldering" V 6030 3350 30  0001 C CNN
+F 2 "SMD_Packages:SMD-0805" V 6030 3350 30  0001 C CNN
 F 3 "" H 6100 3350 30  0000 C CNN
 	1    6100 3350
@@
 F 0 "R303" V 6180 4150 50  0000 C CNN
 F 1 "1K" V 6107 4151 50  0000 C CNN
-F 2 "Resistors_SMD:R_0603_HandSoldering" V 6030 4150 30  0001 C CNN
+F 2 "SMD_Packages:SMD-0805" V 6030 4150 30  0001 C CNN
 F 3 "" H 6100 4150 30  0000 C CNN
 	1    6100 4150

Commit message: Updated the POT references and schematic
Parts:
- R302: value R -> 28.7K
- RV301: value POT -> 10K; footprint Potentiometers:Potentiometer_WirePads_largePads -> CSOS Local:P090L-02F25BR10K
Connections:
- net labels added: 0-2v
- wire segments 21 -> 20
Other:
- moved on the sheet: R302, RV301
Changed lines of the file:
@@
 L R R302
 U 1 1 54E3B0B9
-P 4150 3550
-F 0 "R302" V 4230 3550 50  0000 C CNN
-F 1 "R" V 4157 3551 50  0000 C CNN
-F 2 "SMD_Packages:SMD-0805" V 4080 3550 30  0001 C CNN
-F 3 "" H 4150 3550 30  0000 C CNN
-	1    4150 3550
+P 4300 2850
+F 0 "R302" V 4380 2850 50  0000 C CNN
+F 1 "28.7K" V 4307 2851 50  0000 C CNN
+F 2 "SMD_Packages:SMD-0805" V 4230 2850 30  0001 C CNN
+F 3 "" H 4300 2850 30  0000 C CNN
+	1    4300 2850
 	1    0    0    -1
 $EndComp
@@
 $EndComp
 Wire Wire Line
-	4150 3100 4150 3300
+	4300 3550 4600 3550
 Wire Wire Line
-	4150 3800 4150 4550
+	4300 3100 4300 3550
 Wire Wire Line
 	5400 3150 5400 3250
@@
 L POT RV301
 U 1 1 54E3B0DA
-P 4150 2850
-F 0 "RV301" H 4150 2750 50  0000 C CNN
-F 1 "POT" H 4150 2850 50  0000 C CNN
-F 2 "Potentiometers:Potentiometer_WirePads_largePads" H 4150 2850 60  0001 C CNN
-F 3 "" H 4150 2850 60  0000 C CNN
-	1    4150 2850
+P 4150 3550
+F 0 "RV301" H 4150 3450 50  0000 C CNN
+F 1 "10K" H 4150 3550 50  0000 C CNN
+F 2 "CSOS Local:P090L-02F25BR10K" H 4150 3550 60  0001 C CNN
+F 3 "" H 4150 3550 60  0000 C CNN
+	1    4150 3550
 	0    1    1    0
 $EndComp
 Wire Wire Line
-	4400 2850 4300 2850
-Wire Wire Line
-	4400 1750 4400 2850
+	4300 1750 4300 2600
 Wire Wire Line
 	5400 1750 5400 2350
 Wire Wire Line
 	3900 1750 5400 1750
-Connection ~ 4400 1750
+Connection ~ 4300 1750
 Wire Wire Line
 	5000 1850 5000 1750
@@
 	5000 2650 4600 2650
 Wire Wire Line
-	4600 2650 4600 3200
-Wire Wire Line
-	4600 3200 4150 3200
-Connection ~ 4150 3200
+	4600 2650 4600 3550
 Wire Wire Line
 	6000 2750 6250 2750
@@
 Text GLabel 3900 1750 0    60   Input ~ 0
 2.7V
+Wire Wire Line
+	4150 4550 4150 3800
+Text Label 4650 2650 0    60   ~ 0
+0-2v
 $EndSCHEMATC

Commit message: First cut of layout in preperation for the final session
Parts:
- C301: footprint SMD_Packages:SMD-0805 -> (none)
Connections:
- net labels added: 0-20v
- no-connect marks 0 -> 1
Changed lines of the file:
@@
-	1    0    0    -1
-$EndComp
-$Comp
-L GND #PWR05
-U 1 1 54E3B0C7
-P 5400 3250
-F 0 "#PWR05" H 5400 3000 60  0001 C CNN
-F 1 "GND" H 5400 3100 60  0000 C CNN
-F 2 "" H 5400 3250 60  0000 C CNN
-F 3 "" H 5400 3250 60  0000 C CNN
-	1    5400 3250
-	1    0    0    -1
-$EndComp
-$Comp
-L C C301
-U 1 1 54E3B0CD
-P 5000 2050
-F 0 "C301" H 5050 2150 50  0000 L CNN
-F 1 "C" H 5050 1950 50  0000 L CNN
-F 2 "SMD_Packages:SMD-0805" H 5038 1900 30  0001 C CNN
-F 3 "" H 5000 2050 60  0000 C CNN
-	1    5000 2050
 	1    0    0    -1
 $EndComp
@@
 Wire Wire Line
 	4300 3100 4300 3550
-Wire Wire Line
-	5400 3150 5400 3250
 Wire Wire Line
 	5000 2850 4800 2850
@@
 Connection ~ 5000 1750
 $Comp
-L GND #PWR06
+L GND #PWR05
 U 1 1 54E3B0E8
-P 5000 2350
-F 0 "#PWR06" H 5000 2100 60  0001 C CNN
-F 1 "GND" H 5000 2200 60  0000 C CNN
-F 2 "" H 5000 2350 60  0000 C CNN
-F 3 "" H 5000 2350 60  0000 C CNN
-	1    5000 2350
+P 5000 2300
+F 0 "#PWR05" H 5000 2050 60  0001 C CNN
+F 1 "GND" H 5000 2150 60  0000 C CNN
+F 2 "" H 5000 2300 60  0000 C CNN
+F 3 "" H 5000 2300 60  0000 C CNN
+	1    5000 2300
 	1    0    0    -1
 $EndComp
-Wire Wire Line
-	5000 2350 5000 2250
 Wire Wire Line
 	5000 2650 4600 2650
@@
 Text Label 4650 2650 0    60   ~ 0
 0-2v
+Text Label 5650 3700 0    60   ~ 0
+0-2v
+Text Label 6600 3100 0    60   ~ 0
+0-20v
+NoConn ~ 4150 3300
+Wire Wire Line
+	5400 3150 5400 3250
+Wire Wire Line
+	5000 2250 5000 2300
+$Comp
+L GND #PWR06
+U 1 1 54EE4A9C
+P 5400 3250
+F 0 "#PWR06" H 5400 3000 60  0001 C CNN
+F 1 "GND" H 5400 3100 60  0000 C CNN
+F 2 "" H 5400 3250 60  0000 C CNN
+F 3 "" H 5400 3250 60  0000 C CNN
+	1    5400 3250
+	1    0    0    -1
+$EndComp
+$Comp
+L C C301
+U 1 1 54EE4BC2
+P 5000 2050
+F 0 "C301" H 5050 2150 50  0000 L CNN
+F 1 "C" H 5050 1950 50  0000 L CNN
+F 2 "" H 5038 1900 30  0000 C CNN
+F 3 "" H 5000 2050 60  0000 C CNN
+	1    5000 2050
+	1    0    0    -1
+$EndComp
 $EndSCHEMATC

Commit message: Routing and fixing schematic checkpoint
Parts:
- removed C301: C, symbol C
- U201: footprint SMD_Packages:SOIC-8-N -> (none); MPN LMV358IDR -> (none)
Connections:
- net labels added: 0-2v_FeedBack
- wire segments 20 -> 18
Changed lines of the file:
@@
 $EndDescr
-$Comp
-L LMV358 U201
-U 2 1 54E398B3
-P 5500 2750
-F 0 "U201" H 5450 2950 60  0000 L CNN
-F 1 "LMV358" H 5450 2500 60  0000 L CNN
-F 2 "SMD_Packages:SOIC-8-N" H 5500 2750 60  0001 C CNN
-F 3 "http://www.produktinfo.conrad.com/datenblaetter/1000000-1099999/001072383-da-01-en-IC_OPAMP_GP_R_R_1MH_LMV358IDR_SOIC_8_TID.pdf" H 5500 2750 60  0001 C CNN
-F 4 "LMV358IDR" H 5500 2750 60  0001 C CNN "MPN"
-	2    5500 2750
-	1    0    0    -1
-$EndComp
 $Comp
 L DIODE D301
@@
 	3900 1750 5400 1750
 Connection ~ 4300 1750
-Wire Wire Line
-	5000 1850 5000 1750
-Connection ~ 5000 1750
-$Comp
-L GND #PWR05
-U 1 1 54E3B0E8
-P 5000 2300
-F 0 "#PWR05" H 5000 2050 60  0001 C CNN
-F 1 "GND" H 5000 2150 60  0000 C CNN
-F 2 "" H 5000 2300 60  0000 C CNN
-F 3 "" H 5000 2300 60  0000 C CNN
-	1    5000 2300
-	1    0    0    -1
-$EndComp
 Wire Wire Line
 	5000 2650 4600 2650
@@
 Text Label 4650 2650 0    60   ~ 0
 0-2v
-Text Label 5650 3700 0    60   ~ 0
-0-2v
+Text Label 5200 3700 0    60   ~ 0
+0-2v_FeedBack
 Text Label 6600 3100 0    60   ~ 0
 0-20v
@@
 Wire Wire Line
 	5400 3150 5400 3250
-Wire Wire Line
-	5000 2250 5000 2300
 $Comp
-L GND #PWR06
+L GND #PWR301
 U 1 1 54EE4A9C
 P 5400 3250
-F 0 "#PWR06" H 5400 3000 60  0001 C CNN
+F 0 "#PWR301" H 5400 3000 60  0001 C CNN
 F 1 "GND" H 5400 3100 60  0000 C CNN
 F 2 "" H 5400 3250 60  0000 C CNN
@@
 $EndComp
 $Comp
-L C C301
-U 1 1 54EE4BC2
-P 5000 2050
-F 0 "C301" H 5050 2150 50  0000 L CNN
-F 1 "C" H 5050 1950 50  0000 L CNN
-F 2 "" H 5038 1900 30  0000 C CNN
-F 3 "" H 5000 2050 60  0000 C CNN
-	1    5000 2050
+L LMV358 U201
+U 2 1 54F4A7A0
+P 5500 2750
+F 0 "U201" H 5450 2950 60  0000 L CNN
+F 1 "LMV358" H 5450 2500 60  0000 L CNN
+F 2 "" H 5500 2750 60  0000 C CNN
+F 3 "" H 5500 2750 60  0000 C CNN
+	2    5500 2750
 	1    0    0    -1
 $EndComp

Commit message: Initial route before filling the ground plane
Parts:
- removed U201: LMV358, symbol LMV358
- added U201: LMV358, symbol LMV358
Changed lines of the file:
@@
 	5400 3150 5400 3250
 $Comp
-L GND #PWR301
+L GND #PWR05
 U 1 1 54EE4A9C
 P 5400 3250
-F 0 "#PWR301" H 5400 3000 60  0001 C CNN
+F 0 "#PWR05" H 5400 3000 60  0001 C CNN
 F 1 "GND" H 5400 3100 60  0000 C CNN
 F 2 "" H 5400 3250 60  0000 C CNN
@@
 $Comp
 L LMV358 U201
-U 2 1 54F4A7A0
+U 1 1 54F4A6A3
 P 5500 2750
 F 0 "U201" H 5450 2950 60  0000 L CNN
@@
 F 2 "" H 5500 2750 60  0000 C CNN
 F 3 "" H 5500 2750 60  0000 C CNN
-	2    5500 2750
+F 4 "Value" H 5500 2750 60  0001 C CNN "MPN"
+	1    5500 2750
 	1    0    0    -1
 $EndComp

Commit message: Final update to BOM and added the bom XSL script
Parts:
- D301: value DIODE -> 1N4148
- RV301: MPN (none) -> P090L-02F25BR10K
- U201: MPN Value -> LMV358IDT
Changed lines of the file:
@@
 P 6450 2750
 F 0 "D301" H 6450 2850 50  0000 C CNN
-F 1 "DIODE" H 6450 2650 50  0000 C CNN
+F 1 "1N4148" H 6450 2650 50  0000 C CNN
 F 2 "SMD_Packages:SOD-523" H 6450 2750 60  0001 C CNN
 F 3 "http://www.conrad.de/ce/de/product/1262771/Diode-Fairchild-Semiconductor-1N4148WT-Gehaeuseart-SOD-523-F?ref=searchDetail" H 6450 2750 60  0001 C CNN
@@
 F 2 "CSOS Local:P090L-02F25BR10K" H 4150 3550 60  0001 C CNN
 F 3 "" H 4150 3550 60  0000 C CNN
+F 4 "P090L-02F25BR10K" H 4150 3550 60  0001 C CNN "MPN"
 	1    4150 3550
 	0    1    1    0
@@
 F 2 "" H 5500 2750 60  0000 C CNN
 F 3 "" H 5500 2750 60  0000 C CNN
-F 4 "Value" H 5500 2750 60  0001 C CNN "MPN"
+F 4 "LMV358IDT" H 5500 2750 60  0001 C CNN "MPN"
 	1    5500 2750
 	1    0    0    -1

Commit message: Corrected the default symbol changes in KiCad
Parts:
- D301: symbol DIODE -> D
Connections:
- wire segments 18 -> 19
Changed lines of the file:
@@
 LIBS:valves
 LIBS:CustomComponents
-LIBS:CurrentSinkOrSwim-cache
 EELAYER 25 0
 EELAYER END
@@
 $EndDescr
 $Comp
-L DIODE D301
+L D D301
 U 1 1 54E3AD95
 P 6450 2750
@@
 	4300 3550 4600 3550
 Wire Wire Line
-	4300 3100 4300 3550
+	4300 3000 4300 3550
 Wire Wire Line
 	5000 2850 4800 2850
@@
 $EndComp
 Wire Wire Line
-	4300 1750 4300 2600
+	4300 1750 4300 2700
 Wire Wire Line
 	5400 1750 5400 2350
@@
 	4600 2650 4600 3550
 Wire Wire Line
-	6000 2750 6250 2750
+	6000 2750 6300 2750
 Wire Wire Line
-	6650 2750 7250 2750
+	6600 2750 7250 2750
 $Comp
 L R R301
@@
 $EndComp
 Wire Wire Line
-	6100 4400 6100 4550
+	6100 4300 6100 4550
 Wire Wire Line
 	4150 4550 7250 4550
@@
 	4800 3700 6100 3700
 Wire Wire Line
-	6100 3600 6100 3900
+	6100 3500 6100 4000
 Connection ~ 6100 3700
 Wire Wire Line
@@
 	1    0    0    -1
 $EndComp
+Wire Wire Line
+	6100 3100 6100 3200
 $EndSCHEMATC
