File: VoltageControl.sch (KiCad schematic (older format))
At the start: 6 parts, among them U201 LMV358

Commit message: Added some test results
Parts:
- R302: value 28.7K -> 4k7
Changed lines of the file:
@@
 LIBS:valves
 LIBS:CustomComponents
+LIBS:CurrentSinkOrSwim-cache
 EELAYER 25 0
 EELAYER END
@@
 P 4300 2850
 F 0 "R302" V 4380 2850 50  0000 C CNN
-F 1 "28.7K" V 4307 2851 50  0000 C CNN
+F 1 "4k7" V 4307 2851 50  0000 C CNN
 F 2 "SMD_Packages:SMD-0805" V 4230 2850 30  0001 C CNN
 F 3 "" H 4300 2850 30  0000 C CNN
