File: CurrentControl.sch (KiCad schematic (older format))
At the start: 8 parts, among them P201 HEATSINK, Q201 BUK9575, U201 LMV358

Commit message: Corrected the default symbol changes in KiCad
Parts:
- removed Q201: BUK9575, Transistors_TO-220:TO-220_FET-GDS_Vertical, symbol MOSFET_N
- added Q201: BUK9575, Transistors_TO-220:TO-220_FET-GDS_Vertical, symbol Q_NMOS_GDS
Connections:
- wire segments 22 -> 23
Changed lines of the file:
@@
 LIBS:valves
 LIBS:CustomComponents
-LIBS:CurrentSinkOrSwim-cache
 EELAYER 25 0
 EELAYER END
@@
 $EndComp
 $Comp
-L MOSFET_N Q201
-U 1 1 54E393A3
-P 6550 3000
-F 0 "Q201" H 6560 3170 50  0000 R CNN
-F 1 "BUK9575" H 6500 2850 50  0000 R CNN
-F 2 "Transistors_TO-220:TO-220_FET-GDS_Vertical" H 6550 3000 60  0001 C CNN
-F 3 "" H 6550 3000 60  0000 C CNN
-F 4 "BUK9575-100A,127" H 6550 3000 60  0001 C CNN "MPN"
-	1    6550 3000
-	1    0    0    -1
-$EndComp
-$Comp
 L GND #PWR03
 U 1 1 54E393AA
@@
 $EndComp
 Wire Wire Line
-	6650 3200 6650 4100
+	6650 3200 6650 4200
 Wire Wire Line
 	3200 3350 3650 3350
 Wire Wire Line
-	3200 3350 3200 3550
+	3200 3250 3200 3550
 Wire Wire Line
 	3850 3950 6650 3950
@@
 $EndComp
 Wire Wire Line
-	3200 2000 3200 2850
+	3200 2000 3200 2950
 Wire Wire Line
 	4450 2000 4450 2600
@@
 Connection ~ 3200 2000
 Wire Wire Line
-	4050 2100 4050 2000
+	4050 2000 4050 2150
 Connection ~ 4050 2000
 $Comp
@@
 $EndComp
 Wire Wire Line
-	4050 2600 4050 2500
+	4050 2450 4050 2600
 Wire Wire Line
 	4050 2900 3650 2900
@@
 $EndComp
 Wire Wire Line
-	5050 3000 5400 3000
+	5050 3000 5500 3000
 Wire Wire Line
-	5900 3000 6350 3000
+	5800 3000 6350 3000
 Wire Wire Line
 	6100 3000 6100 1650
@@
 	1    0    0    -1
 $EndComp
+$Comp
+L Q_NMOS_GDS Q201
+U 1 1 551A5476
+P 6550 3000
+F 0 "Q201" H 6850 3050 50  0000 R CNN
+F 1 "BUK9575" H 6600 2800 50  0000 R CNN
+F 2 "Transistors_TO-220:TO-220_FET-GDS_Vertical" H 6750 3100 29  0001 C CNN
+F 3 "" H 6550 3000 60  0000 C CNN
+F 4 "BUK9575-100A,127" H 6550 3000 60  0001 C CNN "MPN"
+	1    6550 3000
+	1    0    0    -1
+$EndComp
+Wire Wire Line
+	6650 4500 6650 4600
+Connection ~ 3200 3350
 $EndSCHEMATC
