File: CurrentControl.sch (KiCad schematic (older format))
At the start: 8 parts, among them P201 HEATSINK, Q201 BUK9575, U201 LMV358

Commit message: Parts update
Parts:
- Q201: footprint Transistors_TO-220:TO-220_FET-GDS_Vertical -> TO_SOT_Packages_THT:TO-220-3_Vertical
Changed lines of the file:
@@
 AR Path="/54E78AC3" Ref="P201"  Part="1"
 AR Path="/54E38472/54E78AC3" Ref="P201"  Part="1"
-F 0 "P201" H 7300 3100 50  0000 C CNN
+F 0 "P201" H 7250 3100 50  0000 C CNN
 F 1 "HEATSINK" V 7400 3000 50  0000 C CNN
 F 2 "CSOS Local:FA-220-38E" H 7300 3000 60  0001 C CNN
@@
 U 1 1 551A5476
 P 6550 3000
-F 0 "Q201" H 6850 3050 50  0000 R CNN
+F 0 "Q201" H 6950 3050 50  0000 R CNN
 F 1 "BUK9575" H 6600 2800 50  0000 R CNN
-F 2 "Transistors_TO-220:TO-220_FET-GDS_Vertical" H 6750 3100 29  0001 C CNN
+F 2 "TO_SOT_Packages_THT:TO-220-3_Vertical" H 6750 3100 29  0001 C CNN
 F 3 "" H 6550 3000 60  0000 C CNN
 F 4 "BUK9575-100A,127" H 6550 3000 60  0001 C CNN "MPN"
