File: PowerRegulation.sch (KiCad schematic (older format))
At the start: 6 parts

Commit message: Initial annotation
Parts:
- R401, R402, R403: renamed from R?; footprint (none) -> Resistors_SMD:R_0603_HandSoldering
- U401: renamed from U?; footprint (none) -> Power_Integrations:SO-8; MPN (none) -> Value
- gave numbers to parts that had none: 2
Connections:
- wire segments 28 -> 18
Changed lines of the file:
@@
 $EndDescr
 $Comp
-L C C?
+L C C401
 U 1 1 54E39CB0
 P 4150 2900
-F 0 "C?" H 4200 3000 50  0000 L CNN
+F 0 "C401" H 4200 3000 50  0000 L CNN
 F 1 "C" H 4200 2800 50  0000 L CNN
-F 2 "" H 4188 2750 30  0000 C CNN
+F 2 "" H 4188 2750 30  0001 C CNN
 F 3 "" H 4150 2900 60  0000 C CNN
 	1    4150 2900
@@
 $EndComp
 $Comp
-L C C?
+L C C402
 U 1 1 54E39CB7
 P 6200 2900
-F 0 "C?" H 6250 3000 50  0000 L CNN
+F 0 "C402" H 6250 3000 50  0000 L CNN
 F 1 "C" H 6250 2800 50  0000 L CNN
-F 2 "" H 6238 2750 30  0000 C CNN
+F 2 "" H 6238 2750 30  0001 C CNN
 F 3 "" H 6200 2900 60  0000 C CNN
 	1    6200 2900
@@
 $EndComp
 $Comp
-L R R?
+L R R402
 U 1 1 54E39CC5
 P 4450 3250
-F 0 "R?" V 4530 3250 50  0000 C CNN
+F 0 "R402" V 4530 3250 50  0000 C CNN
 F 1 "0" V 4457 3251 50  0000 C CNN
-F 2 "" V 4380 3250 30  0000 C CNN
+F 2 "Resistors_SMD:R_0603_HandSoldering" V 4380 3250 30  0001 C CNN
 F 3 "" H 4450 3250 30  0000 C CNN
 F 4 "Value" H 4450 3250 60  0001 C CNN "MPN"
@@
 $EndComp
 Wire Wire Line
-	5500 2550 6200 2550
-Wire Wire Line
-	6200 2550 6950 2550
+	5500 2550 6950 2550
 Wire Wire Line
 	4150 3850 4150 3100
@@
 	6200 3850 6200 3100
 Wire Wire Line
-	4150 3850 4450 3850
-Wire Wire Line
-	4450 3850 5000 3850
-Wire Wire Line
-	5000 3850 5100 3850
-Wire Wire Line
-	5100 3850 5200 3850
-Wire Wire Line
-	5200 3850 5300 3850
-Wire Wire Line
-	5300 3850 5850 3850
-Wire Wire Line
-	5850 3850 6200 3850
+	4150 3850 6200 3850
 Wire Wire Line
 	4450 3500 4450 3850
 $Comp
-L LM2931D-R U?
+L LM2931D-R U401
 U 1 1 54E39CD7
 P 5150 2800
-F 0 "U?" H 5400 2500 60  0000 C CNN
+F 0 "U401" H 5400 2500 60  0000 C CNN
 F 1 "LM2931D-R" H 5150 3200 60  0000 C CNN
-F 2 "" H 5150 2800 60  0000 C CNN
+F 2 "Power_Integrations:SO-8" H 5150 2800 60  0001 C CNN
 F 3 "" H 5150 2800 60  0000 C CNN
+F 4 "Value" H 5150 2800 60  0001 C CNN "MPN"
 	1    5150 2800
 	1    0    0    -1
@@
 	5200 3250 5200 3850
 Wire Wire Line
-	5100 3250 5100 3850
-Wire Wire Line
-	5100 3850 5100 3950
+	5100 3250 5100 3950
 Connection ~ 5100 3850
 $Comp
-L R R?
+L R R401
 U 1 1 54E39CEA
 P 5850 2800
-F 0 "R?" V 5930 2800 50  0000 C CNN
+F 0 "R401" V 5930 2800 50  0000 C CNN
 F 1 "27k" V 5857 2801 50  0000 C CNN
-F 2 "" V 5780 2800 30  0000 C CNN
+F 2 "Resistors_SMD:R_0603_HandSoldering" V 5780 2800 30  0001 C CNN
 F 3 "" H 5850 2800 30  0000 C CNN
 	1    5850 2800
@@
 $EndComp
 $Comp
-L R R?
+L R R403
 U 1 1 54E39CF1
 P 5850 3450
-F 0 "R?" V 5930 3450 50  0000 C CNN
+F 0 "R403" V 5930 3450 50  0000 C CNN
 F 1 "21.6k" V 5857 3451 50  0000 C CNN
-F 2 "" V 5780 3450 30  0000 C CNN
+F 2 "Resistors_SMD:R_0603_HandSoldering" V 5780 3450 30  0001 C CNN
 F 3 "" H 5850 3450 30  0000 C CNN
 	1    5850 3450
@@
 $EndComp
 Wire Wire Line
-	5850 3050 5850 3150
-Wire Wire Line
-	5850 3150 5850 3200
+	5850 3050 5850 3200
 Wire Wire Line
 	5850 3700 5850 3850
@@
 	4450 2700 4700 2700
 Wire Wire Line
-	3750 2550 4150 2550
-Wire Wire Line
-	4150 2550 4700 2550
+	3750 2550 4700 2550
 Wire Wire Line
 	4150 2550 4150 2700

Commit message: Preliminary footprint association
Parts:
- C401, C402: footprint (none) -> SMD_Packages:SMD-0805
- R401, R402, R403: footprint Resistors_SMD:R_0603_HandSoldering -> SMD_Packages:SMD-0805
- U401: footprint Power_Integrations:SO-8 -> SMD_Packages:SOIC-8-N; MPN Value -> LM2931D-R
Changed lines of the file:
@@
 F 0 "C401" H 4200 3000 50  0000 L CNN
 F 1 "C" H 4200 2800 50  0000 L CNN
-F 2 "" H 4188 2750 30  0001 C CNN
+F 2 "SMD_Packages:SMD-0805" H 4188 2750 30  0001 C CNN
 F 3 "" H 4150 2900 60  0000 C CNN
 	1    4150 2900
@@
 F 0 "C402" H 6250 3000 50  0000 L CNN
 F 1 "C" H 6250 2800 50  0000 L CNN
-F 2 "" H 6238 2750 30  0001 C CNN
+F 2 "SMD_Packages:SMD-0805" H 6238 2750 30  0001 C CNN
 F 3 "" H 6200 2900 60  0000 C CNN
 	1    6200 2900
@@
 F 0 "R402" V 4530 3250 50  0000 C CNN
 F 1 "0" V 4457 3251 50  0000 C CNN
-F 2 "Resistors_SMD:R_0603_HandSoldering" V 4380 3250 30  0001 C CNN
+F 2 "SMD_Packages:SMD-0805" V 4380 3250 30  0001 C CNN
 F 3 "" H 4450 3250 30  0000 C CNN
 F 4 "Value" H 4450 3250 60  0001 C CNN "MPN"
@@
 F 0 "U401" H 5400 2500 60  0000 C CNN
 F 1 "LM2931D-R" H 5150 3200 60  0000 C CNN
-F 2 "Power_Integrations:SO-8" H 5150 2800 60  0001 C CNN
-F 3 "" H 5150 2800 60  0000 C CNN
-F 4 "Value" H 5150 2800 60  0001 C CNN "MPN"
+F 2 "SMD_Packages:SOIC-8-N" H 5150 2800 60  0001 C CNN
+F 3 "http://www.produktinfo.conrad.com/datenblaetter/1100000-1199999/001185847-da-01-en-IC_REG_LDO_ADJ_0_1A_LM2931D_R_SOIC_8_STM.pdf" H 5150 2800 60  0001 C CNN
+F 4 "LM2931D-R" H 5150 2800 60  0001 C CNN "MPN"
 	1    5150 2800
 	1    0    0    -1
@@
 F 0 "R401" V 5930 2800 50  0000 C CNN
 F 1 "27k" V 5857 2801 50  0000 C CNN
-F 2 "Resistors_SMD:R_0603_HandSoldering" V 5780 2800 30  0001 C CNN
+F 2 "SMD_Packages:SMD-0805" V 5780 2800 30  0001 C CNN
 F 3 "" H 5850 2800 30  0000 C CNN
 	1    5850 2800
@@
 F 0 "R403" V 5930 3450 50  0000 C CNN
 F 1 "21.6k" V 5857 3451 50  0000 C CNN
-F 2 "Resistors_SMD:R_0603_HandSoldering" V 5780 3450 30  0001 C CNN
+F 2 "SMD_Packages:SMD-0805" V 5780 3450 30  0001 C CNN
 F 3 "" H 5850 3450 30  0000 C CNN
 	1    5850 3450

Commit message: First cut of layout in preperation for the final session
Connections:
- wire segments 18 -> 19
Other:
- moved on the sheet: R401
Changed lines of the file:
@@
 $EndComp
-Wire Wire Line
-	5500 2550 6950 2550
 Wire Wire Line
 	4150 3850 4150 3100
@@
 L R R401
 U 1 1 54E39CEA
-P 5850 2800
-F 0 "R401" V 5930 2800 50  0000 C CNN
-F 1 "27k" V 5857 2801 50  0000 C CNN
-F 2 "SMD_Packages:SMD-0805" V 5780 2800 30  0001 C CNN
-F 3 "" H 5850 2800 30  0000 C CNN
-	1    5850 2800
+P 5850 2850
+F 0 "R401" V 5930 2850 50  0000 C CNN
+F 1 "27k" V 5857 2851 50  0000 C CNN
+F 2 "SMD_Packages:SMD-0805" V 5780 2850 30  0001 C CNN
+F 3 "" H 5850 2850 30  0000 C CNN
+	1    5850 2850
 	-1   0    0    -1
 $EndComp
@@
 $EndComp
 Wire Wire Line
-	5850 3050 5850 3200
+	5850 3100 5850 3200
 Wire Wire Line
 	5850 3700 5850 3850
@@
 	4450 2700 4700 2700
 Wire Wire Line
-	3750 2550 4700 2550
-Wire Wire Line
 	4150 2550 4150 2700
 Connection ~ 4150 2550
 Text GLabel 6950 2550 2    60   Input ~ 0
 2.7V
-Text HLabel 3750 2550 0    60   Input ~ 0
+Text HLabel 3700 2550 0    60   Input ~ 0
 Vin
 Connection ~ 5000 3850
 Connection ~ 5200 3850
 Connection ~ 5300 3850
+Wire Wire Line
+	5850 2550 5850 2600
+Connection ~ 5850 2550
+Wire Wire Line
+	5600 2550 6950 2550
+Wire Wire Line
+	3700 2550 4700 2550
 $EndSCHEMATC

Commit message: Routing and fixing schematic checkpoint
Changed lines of the file:
@@
 $EndComp
 $Comp
-L GND #PWR07
+L GND #PWR401
 U 1 1 54E39CBE
 P 5100 3950
-F 0 "#PWR07" H 5100 3700 60  0001 C CNN
+F 0 "#PWR401" H 5100 3700 60  0001 C CNN
 F 1 "GND" H 5100 3800 60  0000 C CNN
 F 2 "" H 5100 3950 60  0000 C CNN
@@
 Connection ~ 5850 3850
 Wire Wire Line
-	5600 2700 5600 3150
-Wire Wire Line
 	5600 3150 5850 3150
 Connection ~ 5850 3150
@@
 Wire Wire Line
 	3700 2550 4700 2550
+Wire Wire Line
+	5600 3150 5600 2700
 $EndSCHEMATC

Commit message: Final update to BOM and added the bom XSL script
Parts:
- C401, C402: value C -> 0.1uF
- R402: MPN Value -> (none)
Changed lines of the file:
@@
 P 4150 2900
 F 0 "C401" H 4200 3000 50  0000 L CNN
-F 1 "C" H 4200 2800 50  0000 L CNN
+F 1 "0.1uF" H 4200 2800 50  0000 L CNN
 F 2 "SMD_Packages:SMD-0805" H 4188 2750 30  0001 C CNN
 F 3 "" H 4150 2900 60  0000 C CNN
@@
 P 6200 2900
 F 0 "C402" H 6250 3000 50  0000 L CNN
-F 1 "C" H 6250 2800 50  0000 L CNN
+F 1 "0.1uF" H 6250 2800 50  0000 L CNN
 F 2 "SMD_Packages:SMD-0805" H 6238 2750 30  0001 C CNN
 F 3 "" H 6200 2900 60  0000 C CNN
@@
 F 2 "SMD_Packages:SMD-0805" V 4380 3250 30  0001 C CNN
 F 3 "" H 4450 3250 30  0000 C CNN
-F 4 "Value" H 4450 3250 60  0001 C CNN "MPN"
 	1    4450 3250
 	-1   0    0    -1

Commit message: Corrected the default symbol changes in KiCad
Changed lines of the file:
@@
 LIBS:valves
 LIBS:CustomComponents
-LIBS:CurrentSinkOrSwim-cache
 EELAYER 25 0
 EELAYER END
@@
 $EndComp
 Wire Wire Line
-	4150 3850 4150 3100
+	4150 3050 4150 3850
 Wire Wire Line
-	6200 2550 6200 2700
+	6200 2550 6200 2750
 Connection ~ 6200 2550
 Wire Wire Line
-	6200 3850 6200 3100
+	6200 3050 6200 3850
 Wire Wire Line
-	4150 3850 6200 3850
+	6200 3850 4150 3850
 Wire Wire Line
-	4450 3500 4450 3850
+	4450 3400 4450 3850
 $Comp
 L LM2931D-R U401
@@
 $EndComp
 Wire Wire Line
-	5850 3100 5850 3200
+	5850 3000 5850 3300
 Wire Wire Line
-	5850 3700 5850 3850
+	5850 3600 5850 3850
 Connection ~ 5850 3850
 Wire Wire Line
@@
 Connection ~ 4450 3850
 Wire Wire Line
-	4450 3000 4450 2700
+	4450 2700 4450 3100
 Wire Wire Line
 	4450 2700 4700 2700
 Wire Wire Line
-	4150 2550 4150 2700
+	4150 2550 4150 2750
 Connection ~ 4150 2550
 Text GLabel 6950 2550 2    60   Input ~ 0
@@
 Connection ~ 5300 3850
 Wire Wire Line
-	5850 2550 5850 2600
+	5850 2550 5850 2700
 Connection ~ 5850 2550
 Wire Wire Line
