File: CurrentSinkOrSwim.kicad_pcb (KiCad board)
At the start: 2 copper layers, 51.7 x 61.4 mm, 25 parts, among them P101 CONN_01X03, P102 CONN_01X02, P103 CONN_01X02, P201 HEATSINK, U201 LMV358, U401 LM2931D-R

Commit message: Parts update
Parts:
- removed REF** (x4): MountingHole_3mm, CSOS Local:MountingHole_3mm
- added Q201: BUK9575, TO_SOT_Packages_THT:TO-220-3_Vertical, F.Cu at (114.3, 58.6)
Changed lines of the file:
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@@
-(kicad_pcb (version 4) (host pcbnew 0.201508140901+6091~28~ubuntu14.04.1-product)
+(kicad_pcb (version 20171130) (host pcbnew "(5.1.5)-3")
   (general
-    (links 42)
-    (no_connects 0)
-    (area 86.385914 33.1482 147.294086 101.3298)
     (thickness 1.6)
     (drawings 12)
-    (tracks 136)
+    (tracks 135)
     (zones 0)
-    (modules 27)
-    (nets 17)
+    (modules 22)
+    (nets 15)
   )
   (page A4)
@@
     (add_net "Net-(R401-Pad2)")
     (add_net "Net-(R402-Pad1)")
+    (add_net "Net-(RV201-Pad3)")
+    (add_net "Net-(RV301-Pad1)")
   )
   (net_class Power ""
@@
     (add_net GND)
     (add_net "Net-(P101-Pad1)")
+  )
+  (module TO_SOT_Packages_THT:TO-220-3_Vertical (layer F.Cu)
+    (at 114.27 58.59)
+    (descr "TO-220-3, Vertical, RM 2.54mm")
+    (tags "TO-220-3 Vertical RM 2.54mm")
+    (fp_text reference Q201 (at 2.54 -3.62) (layer F.SilkS)
+      (effects (font (size 1 1) (thickness 0.15)))
+    )
+    (fp_text value BUK9575 (at 2.54 3.92) (layer F.Fab)
+      (effects (font (size 1 1) (thickness 0.15)))
+    )
+    (fp_text user %R (at 2.54 -3.62) (layer F.Fab)
+      (effects (font (size 1 1) (thickness 0.15)))
+    )
+    (fp_line (start -2.46 -2.5) (end -2.46 1.9) (layer F.Fab) (width 0.1))
+    (fp_line (start -2.46 1.9) (end 7.54 1.9) (layer F.Fab) (width 0.1))
+    (fp_line (start 7.54 1.9) (end 7.54 -2.5) (layer F.Fab) (width 0.1))
+    (fp_line (start 7.54 -2.5) (end -2.46 -2.5) (layer F.Fab) (width 0.1))
+    (fp_line (start -2.46 -1.23) (end 7.54 -1.23) (layer F.Fab) (width 0.1))
+    (fp_line (start 0.69 -2.5) (end 0.69 -1.23) (layer F.Fab) (width 0.1))
+    (fp_line (start 4.39 -2.5) (end 4.39 -1.23) (layer F.Fab) (width 0.1))
+    (fp_line (start -2.58 -2.62) (end 7.66 -2.62) (layer F.SilkS) (width 0.12))
+    (fp_line (start -2.58 2.021) (end 7.66 2.021) (layer F.SilkS) (width 0.12))
+    (fp_line (start -2.58 -2.62) (end -2.58 2.021) (layer F.SilkS) (width 0.12))
+    (fp_line (start 7.66 -2.62) (end 7.66 2.021) (layer F.SilkS) (width 0.12))
+    (fp_line (start -2.58 -1.11) (end 7.66 -1.11) (layer F.SilkS) (width 0.12))
+    (fp_line (start 0.69 -2.62) (end 0.69 -1.11) (layer F.SilkS) (width 0.12))
+    (fp_line (start 4.391 -2.62) (end 4.391 -1.11) (layer F.SilkS) (width 0.12))
+    (fp_line (start -2.71 -2.75) (end -2.71 2.16) (layer F.CrtYd) (width 0.05))
+    (fp_line (start -2.71 2.16) (end 7.79 2.16) (layer F.CrtYd) (width 0.05))
+    (fp_line (start 7.79 2.16) (end 7.79 -2.75) (layer F.CrtYd) (width 0.05))
+    (fp_line (start 7.79 -2.75) (end -2.71 -2.75) (layer F.CrtYd) (width 0.05))
+    (pad 1 thru_hole rect (at 0 0) (size 1.8 1.8) (drill 1) (layers *.Cu *.Mask)
+      (net 4 "/Current Control/FET_GATE"))
+    (pad 2 thru_hole oval (at 2.54 0) (size 1.8 1.8) (drill 1) (layers *.Cu *.Mask)
+      (net 6 "/Current Control/Current_Sink+"))
+    (pad 3 thru_hole oval (at 5.08 0) (size 1.8 1.8) (drill 1) (layers *.Cu *.Mask)
+      (net 14 "Net-(Q201-Pad3)"))
+    (model ${KISYS3DMOD}/TO_SOT_Packages_THT.3dshapes/TO-220_Neutral123_Vertical.wrl
+      (offset (xyz 2.54 0 0))
+      (scale (xyz 0.4 0.4 0.4))
+      (rotate (xyz 0 0 0))
+    )
   )
   (module SMD_Packages:SMD-0805 (layer B.Cu)
@@
     (pad 3 thru_hole circle (at 2.5 0) (size 2 2) (drill 1) (layers *.Cu *.Mask F.SilkS)
       (net 2 GND))
-  )
-  (module "CSOS Local:MountingHole_3mm" (layer F.Cu)
-    (at 93.98 39.878)
-    (fp_text reference REF** (at 0 5) (layer F.SilkS) hide
-      (effects (font (size 1 1) (thickness 0.15)))
-    )
-    (fp_text value MountingHole_3mm (at 0 -5.5) (layer F.Fab) hide
-      (effects (font (size 1 1) (thickness 0.15)))
-    )
-    (fp_line (start 4 -3.5) (end -4 4) (layer Cmts.User) (width 0.15))
-    (fp_line (start -3.5 -3.5) (end 4 4) (layer Cmts.User) (width 0.15))
-    (fp_circle (center 0 0) (end -3 0) (layer Cmts.User) (width 0.15))
-    (pad "" np_thru_hole circle (at 0 0 180) (size 3 3) (drill 3) (layers *.Cu *.Mask F.SilkS))
-  )
-  (module "CSOS Local:MountingHole_3mm" (layer F.Cu)
-    (at 139.7 39.878)
-    (fp_text reference REF** (at 0 5) (layer F.SilkS) hide
-      (effects (font (size 1 1) (thickness 0.15)))
-    )
-    (fp_text value MountingHole_3mm (at 0 -5.5) (layer F.Fab) hide
-      (effects (font (size 1 1) (thickness 0.15)))
-    )
-    (fp_line (start 4 -3.5) (end -4 4) (layer Cmts.User) (width 0.15))
-    (fp_line (start -3.5 -3.5) (end 4 4) (layer Cmts.User) (width 0.15))
-    (fp_circle (center 0 0) (end -3 0) (layer Cmts.User) (width 0.15))
-    (pad "" np_thru_hole circle (at 0 0 180) (size 3 3) (drill 3) (layers *.Cu *.Mask F.SilkS))
-  )
-  (module "CSOS Local:MountingHole_3mm" (layer F.Cu)
-    (at 139.7 95.25)
-    (fp_text reference REF** (at 0 5) (layer F.SilkS) hide
-      (effects (font (size 1 1) (thickness 0.15)))
-    )
-    (fp_text value MountingHole_3mm (at 0 -5.5) (layer F.Fab) hide
-      (effects (font (size 1 1) (thickness 0.15)))
-    )
-    (fp_line (start 4 -3.5) (end -4 4) (layer Cmts.User) (width 0.15))
-    (fp_line (start -3.5 -3.5) (end 4 4) (layer Cmts.User) (width 0.15))
-    (fp_circle (center 0 0) (end -3 0) (layer Cmts.User) (width 0.15))
-    (pad "" np_thru_hole circle (at 0 0 180) (size 3 3) (drill 3) (layers *.Cu *.Mask F.SilkS))
-  )
-  (module "CSOS Local:MountingHole_3mm" (layer F.Cu)
-    (at 93.98 95.25)
-    (fp_text reference REF** (at 0 5) (layer F.SilkS) hide
-      (effects (font (size 1 1) (thickness 0.15)))
-    )
-    (fp_text value MountingHole_3mm (at 0 -5.5) (layer F.Fab) hide
-      (effects (font (size 1 1) (thickness 0.15)))
-    )
-    (fp_line (start 4 -3.5) (end -4 4) (layer Cmts.User) (width 0.15))
-    (fp_line (start -3.5 -3.5) (end 4 4) (layer Cmts.User) (width 0.15))
-    (fp_circle (center 0 0) (end -3 0) (layer Cmts.User) (width 0.15))
-    (pad "" np_thru_hole circle (at 0 0 180) (size 3 3) (drill 3) (layers *.Cu *.Mask F.SilkS))
   )
   (gr_text "Ext | Self" (at 126.492 80.645 90) (layer F.SilkS)
@@
   (segment (start 116.84 56.769) (end 116.84 58.42) (width 0.6096) (layer F.Cu) (net 6))
   (segment (start 134.62 77.0255) (end 134.62 75.565) (width 0.6096) (layer F.Cu) (net 6) (status 10))
-  (segment (start 119.517686 67.257186) (end 116.638814 67.257186) (width 0.6096) (layer F.Cu) (net 14) (status 10))
-  (segment (start 109.22 74.676) (end 105.156 74.676) (width 0.6096) (layer F.Cu) (net 14) (status 20))
-  (segment (start 116.638814 67.257186) (end 109.22 74.676) (width 0.6096) (layer F.Cu) (net 14))
-  (segment (start 119.38 58.42) (end 119.38 67.1195) (width 0.6096) (layer F.Cu) (net 14) (status 20))
-  (segment (start 119.38 67.1195) (end 119.517686 67.257186) (width 0.6096) (layer F.Cu) (net 14) (status 30))
   (segment (start 105.156 73.406) (end 109.22 73.406) (width 0.254) (layer F.Cu) (net 7) (status 10))
   (segment (start 113.538 69.088) (end 113.538 66.4845) (width 0.254) (layer F.Cu) (net 7) (status 20))
@@
   (segment (start 100.33 68.199) (end 109.011 68.199) (width 0.254) (layer F.Cu) (net 13))
   (segment (start 98.806 69.723) (end 98.806 72.136) (width 0.254) (layer F.Cu) (net 13))
+  (segment (start 119.517686 67.257186) (end 116.638814 67.257186) (width 0.6096) (layer F.Cu) (net 14) (status 10))
+  (segment (start 109.22 74.676) (end 105.156 74.676) (width 0.6096) (layer F.Cu) (net 14) (status 20))
+  (segment (start 116.638814 67.257186) (end 109.22 74.676) (width 0.6096) (layer F.Cu) (net 14))
+  (segment (start 119.38 58.42) (end 119.38 67.1195) (width 0.6096) (layer F.Cu) (net 14) (status 20))
+  (segment (start 119.38 67.1195) (end 119.517686 67.257186) (width 0.6096) (layer F.Cu) (net 14) (status 30))
   (zone (net 0) (net_name "") (layer F.Cu) (hatch edge 0.508)
     (connect_pads (clearance 0.508))

Commit message: Board update and corrections
Other:
- board text added: "Extern 5V"
- board text added: "Sink"
- board text removed: "Extern"
- board text removed: "Sink Input"
Changed lines of the file:
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@@
     (add_net "Net-(R401-Pad2)")
     (add_net "Net-(R402-Pad1)")
-    (add_net "Net-(RV201-Pad3)")
-    (add_net "Net-(RV301-Pad1)")
   )
   (net_class Power ""
@@
     (effects (font (size 1.27 1.27) (thickness 0.127)))
   )
-  (gr_text "Sink Input\n" (at 140.716 84.201 90) (layer F.SilkS)
+  (gr_text "Sink\n" (at 141.02 74.47 90) (layer F.SilkS)
     (effects (font (size 1.27 1.27) (thickness 0.127)))
   )
-  (gr_text Extern (at 140.716 74.295 90) (layer F.SilkS)
+  (gr_text "Extern 5V" (at 141.17 84.87 90) (layer F.SilkS)
     (effects (font (size 1.27 1.27) (thickness 0.127)))
   )
@@
   (gr_line (start 142.6972 36.8808) (end 142.6972 98.2472) (angle 90) (layer Edge.Cuts) (width 0.1))
   (gr_line (start 90.9828 36.8808) (end 142.6972 36.8808) (angle 90) (layer Edge.Cuts) (width 0.1))
-  (gr_text "Current Ctrl\n" (at 118.364 94.615) (layer F.SilkS)
+  (gr_text "Current\nCtrl\n" (at 111.81 94.63) (layer F.SilkS)
     (effects (font (size 1.016 1.016) (thickness 0.127)))
   )
-  (gr_text "Voltage Ctrl" (at 103.759 94.488) (layer F.SilkS)
+  (gr_text "Voltage \nCtrl" (at 98.13 94.51) (layer F.SilkS)
     (effects (font (size 1.016 1.016) (thickness 0.127)))
   )
